File: Watersysteem/PCB Design/PCB_Watersysteem/PCB_Watersysteem.kicad_sch (KiCad schematic)
At the start: 69 parts, among them J1 12V ingang, J10 LED Water Level, J11 LED Nutrient Level, J12 Height Nutrients, J13 Height Mixer, J2 TTL Connector, J23 ReferentieProbe, J24 Voedingsstoffen 1, J25 Voedingsstoffen 2, J26 Voedingsstoffen 3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

Commit message: Update PCB
Placing en routing van vermogen, grootste componenten
Parts:
- removed H3: MountingHole_Pad, MountingHole:MountingHole_3.2mm_M3_Pad_TopBottom, symbol Mechanical:MountingHole_Pad
- added H3: MountingHole, MountingHole:MountingHole_3.2mm_M3, symbol Mechanical:MountingHole
Connections:
- net ECHO_MIX: now also U1.12 (IO27); no longer U1.13 (IO14)
- net ECHO_NUT: now also U1.10 (IO25); no longer U1.11 (IO26)
- net ECHO_WATER: now also U1.8 (IO32); no longer U1.9 (IO33)
- net TRIG_MIX: now also U1.13 (IO14); no longer U1.12 (IO27)
- net TRIG_NUT: now also U1.11 (IO26); no longer U1.10 (IO25)
- net TRIG_WATER: now also U1.9 (IO33); no longer U1.8 (IO32)
Changed lines of the file:
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@@
 	(global_label "TRIG_WATER"
 		(shape input)
-		(at 63.5 96.52 0)
+		(at 63.5 99.06 0)
 		(fields_autoplaced yes)
 		(effects
@@
 		)
 		(property "Intersheetrefs" "${INTERSHEET_REFS}"
-			(at 77.4918 96.52 0)
+			(at 77.4918 99.06 0)
 			(effects
 				(font
@@
 	(global_label "ECHO_MIX"
 		(shape input)
-		(at 63.5 66.04 0)
+		(at 63.5 93.98 0)
 		(fields_autoplaced yes)
 		(effects
@@
 		)
 		(property "Intersheetrefs" "${INTERSHEET_REFS}"
-			(at 75.7985 66.04 0)
+			(at 75.7985 93.98 0)
 			(effects
 				(font
@@
 	(global_label "TRIG_NUT"
 		(shape input)
-		(at 63.5 88.9 0)
+		(at 63.5 91.44 0)
 		(fields_autoplaced yes)
 		(effects
@@
 		)
 		(property "Intersheetrefs" "${INTERSHEET_REFS}"
-			(at 75.1938 88.9 0)
+			(at 75.1938 91.44 0)
 			(effects
 				(font
@@
 	(global_label "ECHO_NUT"
 		(shape input)
-		(at 63.5 91.44 0)
+		(at 63.5 88.9 0)
 		(fields_autoplaced yes)
 		(effects
@@
 		)
 		(property "Intersheetrefs" "${INTERSHEET_REFS}"
-			(at 76.1614 91.44 0)
+			(at 76.1614 88.9 0)
 			(effects
 				(font
@@
 	(global_label "TRIG_MIX"
 		(shape input)
-		(at 63.5 93.98 0)
+		(at 63.5 66.04 0)
 		(fields_autoplaced yes)
 		(effects
@@
 		)
 		(property "Intersheetrefs" "${INTERSHEET_REFS}"
-			(at 74.8309 93.98 0)
+			(at 74.8309 66.04 0)
 			(effects
 				(font
@@
 	(global_label "ECHO_WATER"
 		(shape input)
-		(at 63.5 99.06 0)
+		(at 63.5 96.52 0)
 		(fields_autoplaced yes)
 		(effects
@@
 		)
 		(property "Intersheetrefs" "${INTERSHEET_REFS}"
-			(at 78.4594 99.06 0)
+			(at 78.4594 96.52 0)
 			(effects
 				(font
@@
 	)
 	(symbol
-		(lib_id "Mechanical:MountingHole_Pad")
-		(at 276.86 144.78 90)
+		(lib_id "Device:R")
+		(at 92.71 137.16 0)
 		(unit 1)
 		(exclude_from_sim no)
@@
 		(on_board yes)
 		(dnp no)
-		(fields_autoplaced yes)
-		(property "Reference" "H3"
-			(at 275.59 138.43 90)
+		(property "Reference" "R11"
+			(at 93.218 129.54 0)
 			(effects
 				(font
 					(size 1.27 1.27)
 				)
+				(justify left)
 			)
 		)
-		(property "Value" "MountingHole_Pad"
-			(at 275.59 140.97 90)
+		(property "Value" "10k"
+			(at 93.218 132.08 0)
 			(effects
 				(font
 					(size 1.27 1.27)
 				)
+				(justify left)
 			)
 		)
-		(property "Footprint" "MountingHole:MountingHole_3.2mm_M3_Pad_TopBottom"
-			(at 276.86 144.78 0)
+		(property "Footprint" "Resistor_SMD:R_0805_2012Metric_Pad1.20x1.40mm_HandSolder"
+			(at 90.932 137.16 90)
 			(effects
 				(font
@@
 		)
 		(property "Datasheet" "~"
-			(at 276.86 144.78 0)
+			(at 92.71 137.16 0)
 			(effects
 				(font
@@
 			)
 		)
-		(property "Description" "Mounting Hole with connection"
-			(at 276.86 144.78 0)
+		(property "Description" "Resistor"
+			(at 92.71 137.16 0)
 			(effects
 				(font
@@
 			)
 		)
+		(pin "2"
+		)
 		(pin "1"
 		)
@@
 			(project "PCB_Watersysteem"
 				(path "/de0b8b90-8fde-4ab1-b1b1-e85d44454ecd"
-					(reference "H3")
+					(reference "R11")
 					(unit 1)
 				)
@@
 	)
 	(symbol
-		(lib_id "Device:R")
-		(at 92.71 137.16 0)
+		(lib_id "Mechanical:MountingHole")
+		(at 275.59 144.78 0)
 		(unit 1)
 		(exclude_from_sim no)
@@
 		(on_board yes)
 		(dnp no)
-		(property "Reference" "R11"
-			(at 93.218 129.54 0)
+		(fields_autoplaced yes)
+		(property "Reference" "H3"
+			(at 278.13 143.5099 0)
 			(effects
 				(font
@@
 			)
 		)
-		(property "Value" "10k"
-			(at 93.218 132.08 0)
+		(property "Value" "MountingHole"
+			(at 278.13 146.0499 0)
 			(effects
 				(font
@@
 			)
 		)
-		(property "Footprint" "Resistor_SMD:R_0805_2012Metric_Pad1.20x1.40mm_HandSolder"
-			(at 90.932 137.16 90)
+		(property "Footprint" "MountingHole:MountingHole_3.2mm_M3"
+			(at 275.59 144.78 0)
 			(effects
 				(font
@@
 		)
 		(property "Datasheet" "~"
-			(at 92.71 137.16 0)
+			(at 275.59 144.78 0)
 			(effects
 				(font
@@
 			)
 		)
-		(property "Description" "Resistor"
-			(at 92.71 137.16 0)
+		(property "Description" "Mounting Hole without connection"
+			(at 275.59 144.78 0)
 			(effects
 				(font
@@
 			)
 		)
-		(pin "2"
-		)
-		(pin "1"
-		)
 		(instances
-			(project "PCB_Watersysteem"
+			(project ""
 				(path "/de0b8b90-8fde-4ab1-b1b1-e85d44454ecd"
-					(reference "R11")
+					(reference "H3")
 					(unit 1)
 				)
@@
 					(unit 1)
 				)
-			)
-		)
-	)
-	(symbol
-		(lib_id "power:GND")
-		(at 279.4 144.78 0)
-		(unit 1)
-		(exclude_from_sim no)
-		(in_bom yes)
-		(on_board yes)
-		(dnp no)
-		(fields_autoplaced yes)
-		(property "Reference" "#PWR032"
-			(at 279.4 151.13 0)
-			(effects
-				(font
-					(size 1.27 1.27)
-				)
-				(hide yes)
-			)
-		)
-		(property "Value" "GND"
-			(at 279.4 149.86 0)
-			(effects
-				(font
-					(size 1.27 1.27)
-				)
-			)
-		)
-		(property "Footprint" ""
-			(at 279.4 144.78 0)
-			(effects
-				(font
-					(size 1.27 1.27)
-				)
-				(hide yes)
-			)
-		)
-		(property "Datasheet" ""
-			(at 279.4 144.78 0)
-			(effects
-				(font
-					(size 1.27 1.27)
-				)
-				(hide yes)
-			)
-		)
-		(property "Description" "Power symbol creates a global label with name \"GND\" , ground"
-			(at 279.4 144.78 0)
-			(effects
-				(font
-					(size 1.27 1.27)
-				)
-				(hide yes)
-			)
-		)
-		(pin "1"
-		)
-		(instances
-			(project "PCB_Watersysteem"
-				(path "/de0b8b90-8fde-4ab1-b1b1-e85d44454ecd"
-					(reference "#PWR032")
-					(unit 1)
-				)
