File: Watersysteem/PCB Design/PCB_Watersysteem/PCB_Watersysteem.kicad_pcb (KiCad board)
At the start: 2 copper layers, 98 parts, among them J1 12V ingang, J10 LED Water Level, J11 LED Nutrient Level, J12 Height Nutrients, J13 Height Mixer, J14 Pomp1, J15 Pomp2, J16 Pomp3, J17 Pomp4, J18 Luchtpomp, J19 Mixer, J2 TTL Connector, J20 UV, J22 230V, J23 ReferentieProbe, J24 Voedingsstoffen 1, J25 Voedingsstoffen 2, J26 Voedingsstoffen 3, J6 Height Water, J7 Endstop Lade0, J8 Endstop Lade1, J9 Endstop UV, K1 AHQSS105DM2FA0G, K2 AHQSS105DM2FA0G, K3 AHQSS105DM2FA0G, K6 AHQSS105DM2FA0G, K7 AHQSS105DM2FA0G, K8 AHQSS105DM2FA0G, K9 AHQSS105DM2FA0G, Q1 BSS138, Q2 BSS138, Q3 BSS138, Q4 BSS138, Q5 BSS138, Q6 BSS138, Q7 BSS138, SW1 EN, SW2 BOOT, U1 ESP32-WROOM-32D, U2 MP1584_Module, U3 AMS1117-3.3, U4 ADS1115IDGS, U5 MCP23017_SO

Commit message: Update PCB
Start met floorplanning
Parts:
- moved C1 152.0 mm to (93.5, 162.1), turned to 90 degrees
- moved C2 125.0 mm to (123.4, 162.1), turned to 90 degrees
- moved C3 123.1 mm to (131.1, 164.1), turned to 90 degrees
- moved J1 119.2 mm to (73.7, 160.0)
- moved U2 110.6 mm to (108.5, 159.6)
- moved U3 109.6 mm to (137.9, 162.8)
- moved C14 78.7 mm to (187.5, 148.6), turned to 180 degrees
- moved R1 75.5 mm to (154.9, 163.1)
- moved J6 74.1 mm to (269.1, 22.1)
- moved J12 74.1 mm to (273.8, 22.1)
- moved J23 74.1 mm to (203.5, 54.0)
- moved J24 74.1 mm to (220.2, 54.0)
- moved J25 74.1 mm to (237.0, 54.0)
- moved J26 74.1 mm to (253.8, 54.0)
- moved C10 74.1 mm to (269.3, 33.5)
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
Commit message: PCB Design
PCB Design (nog niet volledig af)
Parts:
- added J3: Extra GPIO, Connector_PinHeader_2.54mm:PinHeader_1x06_P2.54mm_Vertical, F.Cu at (158.0, 85.0)
- C10, C11, C12, C14, C4, C5, C6, C8, C9, D1, D10, D11, D12, D13, D7, D8, D9, R10, R11, R12, R13, R3, R4, R6, R7, R8, R9, U3: moved to B.Cu
- moved J13 173.8 mm to (107.8, 55.6), turned to -90 degrees
- moved J12 158.3 mm to (119.0, 55.6), turned to -90 degrees
- moved J6 142.9 mm to (130.3, 55.7), turned to -90 degrees
- moved C7 132.3 mm to (133.4, 60.0), turned to 180 degrees
- moved K9 131.6 mm to (156.6, 111.3), turned to -90 degrees
- moved C5 129.8 mm to (136.4, 57.2), turned to -90 degrees
- moved C6 127.3 mm to (138.4, 57.2), turned to -90 degrees
- moved C8 114.6 mm to (153.9, 75.4), turned to 90 degrees
- moved C12 111.1 mm to (173.4, 95.5), turned to 180 degrees
- moved C11 109.4 mm to (177.2, 95.5)
- moved C10 109.0 mm to (176.2, 90.2)
- moved K8 108.0 mm to (136.9, 111.3), turned to -90 degrees
- moved J2 105.7 mm to (164.3, 55.6), turned to -90 degrees
- moved C13 103.9 mm to (177.2, 90.4)
- moved JP2 101.7 mm to (137.5, 87.9), turned to 0 degrees
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Connections:
- net SCL0 renamed I2C-
- net SDA0 renamed I2C+
- U4 pad 1: GND -> Net-(JP1-B)
- U4 pad 4: Nutr0 -> Nutr3
- U4 pad 5: Nutr1 -> Nutr2
- U4 pad 6: Nutr2 -> Nutr1
- U4 pad 7: Nutr3 -> Nutr0
- U5 pad 1: unconnected-(U5-GPB0-Pad1) -> GPB0
- U5 pad 2: unconnected-(U5-GPB1-Pad2) -> GPB1
- U5 pad 3: unconnected-(U5-GPB2-Pad3) -> GPB2
- U5 pad 4: unconnected-(U5-GPB3-Pad4) -> GPB3
Routing:
- net 3V3: track 0.00 -> 168.8 mm, vias 0 -> 5
- net 5V: track 0.00 -> 166.6 mm
- net 12V: track 0.00 -> 136.1 mm
- net I2C-: track 0.00 -> 63.7 mm, vias 0 -> 2
- net I2C+: track 0.00 -> 62.6 mm, vias 0 -> 2
- net RELAY_PUMP4: track 0.00 -> 47.0 mm
- net ECHO_MIX: track 0.00 -> 39.6 mm
- net RELAY_PUMP3: track 0.00 -> 36.8 mm
- net TRIG_MIX: track 0.00 -> 36.5 mm
- net Nutr3: track 0.00 -> 31.9 mm, vias 0 -> 1
- net Nutr0: track 0.00 -> 31.4 mm, vias 0 -> 1
- net RELAY_UV: track 0.00 -> 28.5 mm
- net ECHO_NUT: track 0.00 -> 27.3 mm
- net RELAY_PUMP2: track 0.00 -> 26.7 mm
- net GPB0: track 0.00 -> 24.8 mm, vias 0 -> 1
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- added copper zone on B.Cu, net GND
- added copper zone on F.Cu, net GND
Other:
- board outline added: 111.5 x 93.5 mm
- board text added: "3V3"
- board text added: "Aan GND van ontkoppelcondensatoren een via indien mogelijk (lagere impedantie naar GND plane)"
- board text added: "ECHO MIX"
- board text added: "ECHO NUT"
- board text added: "ECHO WATER"
- board text added: "END_1"
- board text added: "END_2"
- board text added: "END_3"
- board text added: "GND"
- board text added: "I2C/UART differential tracks maken"
- board text added: "LED_NUT"
- board text added: "LED_WATER"
- board text added: "Mooie spacing traces"
- board text added: "ONDER AC GEEN GROUND PLANE: ISOLEREN"
- board text added: "Opletten dat onder elke trace zo veel mogelijk GND plane zit (dus bv bij via clearance opletten)"
- board text added: "Product nummer pcbway plaats geven: {dblquote}WayWayWay{dblquote} ergens zetten"
- board text added: "TRIG MIX"
- board text added: "TRIG NUT"
- board text added: "TRIG WATER"
