File: Watersysteem/PCB Design/PCB_Watersysteem/relays.kicad_sch (KiCad schematic)
At the start: 29 parts, among them J12 Pomp2, J16 Pomp3, J17 Pomp4, J20 Luchtpomp, J22 Mixer, J23 230V, J24 UV, J6 Pomp1, K1 AHQSS105DM2FA0G, K2 AHQSS105DM2FA0G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

Commit message: Update PCB
Eindwerk aan PCB (extra vias, meer silkscreen, lichte aanpassing floorplanning,...)
Parts:
- removed D10, D4, D5, D6, D7, D8, D9: 1N4148W, Diode_SMD:D_SOD-123, symbol Diode:1N4148W
- added D10, D4, D5, D6, D7, D8, D9: 1N4148, Diode_SMD:D_0805_2012Metric_Pad1.15x1.40mm_HandSolder, symbol Diode:1N4148
Connections:
- net 5V: now also D10.1 (K), D4.1 (K), D5.1 (K), D6.1 (K), D7.1 (K), D8.1 (K), D9.1 (K)
- net at K7.4 (COIL_2), Q7.3 (D): now also D10.2 (A)
- net at K5.4 (COIL_2), Q5.3 (D): now also D8.2 (A)
- net at K4.4 (COIL_2), Q6.3 (D): now also D9.2 (A)
- net at K2.4 (COIL_2), Q2.3 (D): now also D5.2 (A)
- net at K6.4 (COIL_2), Q4.3 (D): now also D7.2 (A)
- net at K1.4 (COIL_2), Q1.3 (D): now also D4.2 (A)
- net at K3.4 (COIL_2), Q3.3 (D): now also D6.2 (A)
